File: halakekit_lino.sch (KiCad schematic (older format))
At the start: 13 parts, among them J1 HEADER_10, U1 MDBT40, U2 NJM2870, U3 RTF015N03, Y1 Crystal

Commit message: Update pcb to rev3.0
Parts:
- C4: footprint Capacitors_SMD:C_1812 -> register_and_condensor:C_0603
Changed lines of the file:
@@
 F 0 "C4" H 7125 5000 50  0000 L CNN
 F 1 "4.7uf1" H 7125 4800 50  0000 L CNN
-F 2 "Capacitors_SMD:C_1812" H 7138 4750 50  0001 C CNN
+F 2 "register_and_condensor:C_0603" H 7138 4750 50  0001 C CNN
 F 3 "" H 7100 4900 50  0000 C CNN
 	1    7100 4900
