File: pcb/halakekit_lino_order.kicad_pcb (KiCad board)
At the start: 2 copper layers, 30.1 x 20.1 mm, 19 parts, among them J1 HEADER_10, U1 MDBT40, U2 NJM2870, U3 RTF015N03, Y1 Crystal

Commit message: Update plot files to order
Parts:
- added BT1: Battery, CR2032_frame:BAT-HLD-001-TRCT, B.Cu at (156.7, 86.9)
- added C1: 12pf, register_and_condensor:C_0603, F.Cu at (167.9, 77.5)
- added C2: 12pf, register_and_condensor:C_0603, F.Cu at (161.3, 77.5)
- added C3: 0.01uf, register_and_condensor:C_0603, F.Cu at (152.2, 77.5)
- added C4: 4.7uf1, register_and_condensor:C_0603, F.Cu at (150.4, 77.5)
- added C5: 0.1uf1, register_and_condensor:C_0603, F.Cu at (159.5, 77.5)
- added G***: LOGO, logos:nyampass_logo_8p4mm, F.Cu at (151.0, 88.8)
- added G***: LOGO, osh-logo:osh-logo-3p4mm, B.Cu at (146.3, 82.1)
- added G***: LOGO, osh-logo:osh-logo-3p4mm, F.Cu at (171.7, 77.2)
- added G***: LOGO, logos:nyampass_logo_8p4mm, B.Cu at (148.6, 77.7)
- added J1: HEADER_10, simple_headers:Pin_Header_Straight_1x10, F.Cu at (168.2, 73.4)
- added R1: 1K, register_and_condensor:R_0603, F.Cu at (157.8, 77.5)
- added R2: 1K, register_and_condensor:R_0603, F.Cu at (148.4, 77.5)
- added U1: MDBT40, MDBT40:MDBT40, F.Cu at (165.1, 84.9)
- added U2: NJM2870, common:SOT-23-5, F.Cu at (155.0, 77.5)
- added U3: RTF015N03, mosfet:rtf015n03, F.Cu at (145.1, 77.5)
- added Y1: Crystal, common:FC-135, F.Cu at (164.6, 77.5)
Routing:
- net +3V3: track 45.3 -> 90.6 mm, vias 2 -> 4
- net GND: track 30.1 -> 60.1 mm, vias 9 -> 18
- net SWDCLK: track 17.8 -> 35.6 mm, vias 1 -> 2
- net SWDIO: track 16.8 -> 33.6 mm, vias 1 -> 2
- net P3: track 16.1 -> 32.2 mm, vias 1 -> 2
- net P0: track 15.9 -> 31.7 mm, vias 1 -> 2
- net P1: track 14.3 -> 28.6 mm, vias 1 -> 2
- net P4: track 14.2 -> 28.4 mm
- net P2: track 13.9 -> 27.7 mm, vias 1 -> 2
- net Net-(C1-Pad1): track 10.4 -> 20.7 mm
- net VCC: track 7.20 -> 14.4 mm
- net Net-(C2-Pad1): track 6.30 -> 12.6 mm
- net Net-(R1-Pad2): track 4.60 -> 9.20 mm, vias 2 -> 4
- net P4_Drain: track 4.17 -> 8.34 mm
- net Net-(C3-Pad1): track 1.78 -> 3.55 mm
Other:
- board size 30.1 x 20.1 mm -> 30.1 x 41 mm
